Commit message: Sensor logic to take the output only from the road point that you are on top of

File: goodbot.urdf (robot description, URDF)
Before this commit: robot robotel2.0, 11 links, 10 joints
Links:
- removed link link_FrontTurn
- removed link link_FrontWheel
- removed link link_LWheel
- removed link link_RWheel
- added link link_FWL, mass 15.0; collision cylinder length=0.2 radius=1.0; visual cylinder length=0.2 radius=1.0
- added link link_FWR, mass 15.0; collision cylinder length=0.2 radius=1.0; visual cylinder length=0.2 radius=1.0
- added link link_RWL, mass 15.0; collision cylinder length=0.2 radius=1.0; visual cylinder length=0.2 radius=1.0
- added link link_RWR, mass 15.0; collision cylinder length=0.2 radius=1.0; visual cylinder length=0.2 radius=1.0
- added link link_Steer, mass 0.01; collision box size=0.24 0.24 0.24; visual box size=0.24 0.24 0.24
- link link_Body: mass 10.0 -> 30.0; geometry collision box size=3.7 2.0 0.6; visual box size=3.7 2.0 0.6
- link link_Sensor1: mass 1.0 -> 3.0
- link link_Sensor2: mass 1.0 -> 3.0
- link link_Sensor3: mass 1.0 -> 3.0
- link link_Sensor4: mass 1.0 -> 3.0
- link link_Sensor5: mass 1.0 -> 3.0
- link link_Sensor6: mass 1.0 -> 3.0
Joints:
- removed joint link_FrontTurn
- removed joint link_FrontWheel
- removed joint link_LWheel
- removed joint link_RWheel
- added joint link_FWL: type continuous, parent link_Steer, child link_FWL, origin xyz=0.10256 1.15192 -0.50406 rpy=1.5708 0 0, axis 0 0 1.0, limit effort=0 velocity=0
- added joint link_FWR: type continuous, parent link_Steer, child link_FWR, origin xyz=0.10256 -1.14808 -0.50406 rpy=1.5708 0 0, axis 0 0 1.0, limit effort=0 velocity=0
- added joint link_RWL: type continuous, parent link_Body, child link_RWL, origin xyz=-1.65 1.15 0 rpy=1.5708 0 0, axis 0 0 1.0, limit effort=0 velocity=0
- added joint link_RWR: type continuous, parent link_Body, child link_RWR, origin xyz=-1.65 -1.15 0 rpy=1.5708 0 0, axis 0 0 1.0, limit effort=0 velocity=0
- added joint link_Steer: type revolute, parent link_Body, child link_Steer, origin xyz=1.44744 -0.00192 0.50406 rpy=0 0 0, axis 0 0 1, limit effort=0 velocity=0
- joint link_Sensor1: origin xyz=2.04744 1.49808 0.32406 rpy=0 0 0 -> xyz=2.94744 1.49808 0.32406 rpy=0 0 0
- joint link_Sensor2: origin xyz=2.04744 0.89808 0.32406 rpy=0 0 0 -> xyz=2.94744 0.89808 0.32406 rpy=0 0 0
- joint link_Sensor3: origin xyz=2.04744 0.29808 0.32406 rpy=0 0 0 -> xyz=2.94744 0.29808 0.32406 rpy=0 0 0
- joint link_Sensor4: origin xyz=2.04744 -0.30192 0.32406 rpy=0 0 0 -> xyz=2.94744 -0.30192 0.32406 rpy=0 0 0
- joint link_Sensor5: origin xyz=2.04744 -0.90192 0.32406 rpy=0 0 0 -> xyz=2.94744 -0.90192 0.32406 rpy=0 0 0
- joint link_Sensor6: origin xyz=2.04744 -1.50192 0.32406 rpy=0 0 0 -> xyz=2.94744 -1.50192 0.32406 rpy=0 0 0
